File: ball_launcher_kicad/ball_launcher_kicad.kicad_sch (KiCad schematic)
At the start: 32 parts, among them J1 Battery 9V, J2 Power Source 12V 2A, J3 STLINK, J4 Proximity Sensor E18-D80NK, M1 Motor DC 50W, Q1 IRF540N, SW1 Button, U1 EA_DOGS104B-A, U2 STM32F411CEUx, U3 LM1117-5.0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

Commit message: Definição do part numbers, criação do BOM e do geber
Parts:
- C1, C14: Manufacturer part number (none) -> C3216X6S2A106K16; Mouser part number (none) -> 810-C3216X6S2A106K16
- C10, C7: Manufacturer part number (none) -> C1206C105K3NAUTO; Mouser part number (none) -> 80-C1206C105K3NAUTO
- C11, C12: Manufacturer part number (none) -> C0805X334K5RACAUTO; Mouser part number (none) -> 80-C0805X334K5RACAUTO
- C13: Manufacturer part number (none) -> C1206X475K4NACAUTO; Mouser part number (none) -> 80-C1206X475K4NACAUTO
- C2, C3, C4, C5, C6, C8: Manufacturer part number (none) -> C0805C104K5RAC7411; Mouser part number (none) -> 80-C0805C104K5RAC7411
- C9: Manufacturer part number (none) -> C2012X5R2A475K12; Mouser part number (none) -> 810-C2012X5R2A475K12
- D1: Manufacturer part number (none) -> 1N4001; Mouser part number (none) -> 637-1N4001
- J1: Manufacturer part number (none) -> 12BH610-GR; Mouser part number (none) -> 12BH610-GR
- J2, M1: Manufacturer part number (none) -> 1711725; Mouser part number (none) -> 651-1711725
- J3: Manufacturer part number (none) -> 3-644456-5; Mouser part number (none) -> 571-3-644456-5
- J4: Manufacturer part number (none) -> 1714735; Mouser part number (none) -> 651-1714735
- L1: Manufacturer part number (none) -> P0850NL; Mouser part number (none) -> 673-P0850NL
- Q1: Manufacturer part number (none) -> STP40NF10L; Mouser part number (none) -> 511-STP40NF10L
- R1, R2: Manufacturer part number (none) -> SDR10EZPJ222; Mouser part number (none) -> 755-SDR10EZPJ222
- R10, R3, R6: Manufacturer part number (none) -> SDR10EZPJ103; Mouser part number (none) -> 755-SDR10EZPJ103
- SW1: Manufacturer part number (none) -> B3S-1000; Mouser part number (none) -> 653-B3S-1000
- U1: Manufacturer part number (none) -> EADOGS104W-A; Mouser part number (none) -> 790-EADOGS104W-A
- U2: Manufacturer part number (none) -> STM32F411CEU6; Mouser part number (none) -> 511-STM32F411CEU6
- U3: Manufacturer part number (none) -> LM1117T-50/NOPB; Mouser part number (none) -> 926-LM1117T-50/NOPB
- U4: Manufacturer part number (none) -> LM1117SX33NOPB; Mouser part number (none) -> 926-LM1117SX33NOPB
